File: hw/stripboard/powerctl.sch (EAGLE design)
At the start: 15 parts, among them J3 JST-B3B-XH, U1 ATTiny85P

Commit message: hw: add PCB hardware definition and CAM files
Parts:
- removed H1, H2: MOUNT-HOLE4.1, holes:MOUNT-HOLE4.1
- removed J6: (no value), pinhead:PINHD-1X3/90
- removed JP1: (no value), pinhead:PINHD-1X3
- removed U1: ATTiny85P, SparkFun:ATTINY85P
- added U$1: ATTINY85-PU, SparkFun:ATTINY13DIP
- J1: device pinhead:PINHD-1X2 -> SparkFun-Connectors:CONN_02
- J2: value (none) -> MA03-2; device pinhead:PINHD-2X3/90 -> pinhead:PINHD-2X3
- J3: value JST-B3B-XH -> JST-XT-3P; device jst-xh:JST-B3B-XH -> SparkFun-Connectors:CONN_03
- J4: device pinhead:PINHD-1X2/90 -> SparkFun-Connectors:CONN_02
- J5: device pinhead:PINHD-1X9 -> SparkFun-Connectors:CONN_02
- R1, R2, R3, R4: device rcl:R-US_0207/7 -> rcl:R-US_0207/15
Connections:
- net LEDBO renamed N$1
- net LEDGO renamed N$3
- net LEDRO renamed N$2
- removed net AC-L: J5.9, J6.1
- removed net AC-N: J5.7, J6.3
- removed net LEDCO: J2.1, JP1.2
- removed net PE: J5.4, J5.5, J5.6, J5.8, J6.2
- net !OFF: now also U$1.PB5(NRES); no longer U1.PB5(!RST!)
- net +5V: now also J2.1, J5.1, U$1.VCC; no longer J5.2, JP1.3, U1.VCC
- net BUTTON: now also U$1.PB3(ADC3); no longer U1.PB3(ADC3)
- net GND: now also J5.2, U$1.GND; no longer J5.1, JP1.1, U1.GND
- net LEDB: now also U$1.PB0(MOSI); no longer U1.PB0(MOSI)
- net LEDG: now also U$1.PB1(MISO); no longer U1.PB1(MISO)
- net LEDR: now also U$1.PB4(ADC2); no longer U1.PB4(ADC2)
- net SSR: now also U$1.PB2(SCK/ADC1); no longer U1.PB2(SCK/ADC1)
Other:
- note added: "From mini PSU module"
- note added: "To pushbutton 1 - LED common (+5V for common anode, GND for common cathode) 2 - Button 3 - Red LED 4 - Green LED 5 - Button 6 - Blue LED"
- note removed: "AC in"
- note removed: "CA CC"
- note removed: "LED polarity"
- note removed: "Mini PSU"
- note removed: "To pushbutton 1 - LED common 2 - Button 3 - Red LED 4 - Green LED 5 - Button 6 - Blue LED"
- moved on the sheet: J1, J4
